File: servo.kicad_pcb (KiCad board)
At the start: 2 copper layers, 28 parts, among them J1 Conn_02x04_Counter_Clockwise, Q1 IL?, Q2 Il?, Q3 Il?, Q4 Il?, U1 ATmega328-AU, U2 LM3480-5.0, U3 ZXCT1009F

Commit message: 'a'
Parts:
- Q1, Q2, Q3, Q4: footprint Package_TO_SOT_SMD:SOT-23 -> Package_TO_SOT_SMD:SOT-223-3_TabPin2
- moved J1 44.6 mm to (171.9, 71.8)
- moved U1 42.6 mm to (126.9, 55.1)
- moved Q2 35.9 mm to (143.4, 69.2), turned to 90 degrees
- moved Q4 32.2 mm to (143.4, 78.3)
- moved Q3 30.5 mm to (151.3, 69.2), turned to 270 degrees
- moved Q1 20.9 mm to (151.4, 78.2)
- moved U3 10.4 mm to (177.6, 87.6)
Routing:
- net GND: track 18.6 -> 0.00 mm
- net Net-(Q1-Pad3): track 13.9 -> 0.00 mm
- net Net-(Q1-Pad1): track 9.49 -> 0.02 mm
- net Net-(Q1-Pad2): track 9.33 -> 0.00 mm
- net Net-(R2-Pad1): track 4.93 -> 0.00 mm
- net Net-(C6-Pad1): track 4.66 -> 0.00 mm
- net /Q2AG: track 4.53 -> 0.00 mm
- net /Q1AG: track 2.23 -> 0.00 mm
Other:
- board outline added: 38 x 18 mm
