File: servo.sch (KiCad schematic (older format))
At the start: 28 parts, among them J1 Conn_02x04_Counter_Clockwise, Q1 IL?, Q2 Il?, Q3 Il?, Q4 Il?, U1 ATmega328-AU, U2 LM3480-5.0, U3 ZXCT1009F

Commit message: 'a'
Parts:
- Q1, Q2, Q3, Q4: footprint Package_TO_SOT_SMD:SOT-23 -> Package_TO_SOT_SMD:SOT-223-3_TabPin2
Changed lines of the file:
@@
 F 0 "Q2" H 9000 2650 50  0000 L CNN
 F 1 "Il?" H 9000 2550 50  0000 L CNN
-F 2 "Package_TO_SOT_SMD:SOT-23" H 8950 2750 50  0001 C CNN
+F 2 "Package_TO_SOT_SMD:SOT-223-3_TabPin2" H 8950 2750 50  0001 C CNN
 F 3 "~" H 8750 2650 50  0001 C CNN
 	1    8750 2650
@@
 F 0 "Q4" H 10150 2650 50  0000 L CNN
 F 1 "Il?" H 10150 2800 50  0000 L CNN
-F 2 "Package_TO_SOT_SMD:SOT-23" H 10100 2750 50  0001 C CNN
+F 2 "Package_TO_SOT_SMD:SOT-223-3_TabPin2" H 10100 2750 50  0001 C CNN
 F 3 "~" H 9900 2650 50  0001 C CNN
 	1    9900 2650
@@
 F 0 "Q3" H 10150 2100 50  0000 L CNN
 F 1 "Il?" H 10100 1950 50  0000 L CNN
-F 2 "Package_TO_SOT_SMD:SOT-23" H 10100 2200 50  0001 C CNN
+F 2 "Package_TO_SOT_SMD:SOT-223-3_TabPin2" H 10100 2200 50  0001 C CNN
 F 3 "~" H 9900 2100 50  0001 C CNN
 	1    9900 2100
@@
 F 0 "Q1" H 9000 2100 50  0000 L CNN
 F 1 "IL?" H 9000 1950 50  0000 L CNN
-F 2 "Package_TO_SOT_SMD:SOT-23" H 8950 2200 50  0001 C CNN
+F 2 "Package_TO_SOT_SMD:SOT-223-3_TabPin2" H 8950 2200 50  0001 C CNN
 F 3 "~" H 8750 2100 50  0001 C CNN
 	1    8750 2100
